File: PCB/9mini.kicad_sch (KiCad schematic)
At the start: 15 parts

Commit message: completing the schematic
Parts:
- added C1, C10, C11, C12, C7, C9: 0.1uF, symbol Device:C
- added C2, C3, C6, C8: 1uF, symbol Device:C
- added C4, C5: 15pF, symbol Device:C
- added D1, D2, D3, D4, D5, D6: WS2812B, LED_SMD:LED_WS2812B_PLCC4_5.0x5.0mm_P3.2mm, symbol LED:WS2812B
- added J1: Conn_01x04, symbol Connector_Generic:Conn_01x04
- added R1, R3, R4: 1K, symbol Device:R
- added R2: NC, symbol Device:R
- added R5, R6: 27R, symbol Device:R
- added SW1, SW2: SW_Push, symbol Switch:SW_Push
- added U1: ~, symbol my_Library:XC6206
- added U2: W25Q16JVUXIQ, symbol my_Library:W25Q16JVUXIQ
- added U3: RP2040, Package_DFN_QFN:QFN-56-1EP_7x7mm_P0.4mm_EP3.2x3.2mm, symbol MCU_RaspberryPi:RP2040
- added Y1: Crystal_GND23, symbol Device:Crystal_GND23
- renumbered MX13 to MX11, MX14 to MX12, MX15 to MX13, MX11 to MX14, MX12 to MX15
Connections:
- net GND: now reaches MX15.1 (COL)
- net GND: now also MX1.1 (COL), MX10.1 (COL), MX11.1 (COL), MX12.1 (COL), MX13.1 (COL), MX14.1 (COL), MX2.1 (COL), MX3.1 (COL), MX4.1 (COL), MX5.1 (COL), MX6.1 (COL), MX7.1 (COL), MX8.1 (COL), MX9.1 (COL), C1.1, C10.1, C11.1, C12.1, C2.2, C3.2, C4.2, C5.2, C6.1, C7.1, C8.1, C9.1, D1.3 (VSS), D2.3 (VSS), D3.3 (VSS), D4.3 (VSS), D5.3 (VSS), D6.3 (VSS), J1.4 (Pin_4), SW1.2, SW2.2, U1.1 (GND), U2.4 (GND), U3.57 (GND), Y1.2, Y1.3
- net SW12: now reaches MX15.2 (ROW)
- net SW12: now also U3.14 (GPIO11)
- net SW3: now reaches MX3.2 (ROW)
- net SW3: now also U3.4 (GPIO2)
- net SW1: now reaches MX1.2 (ROW)
- net SW1: now also U3.2 (GPIO0)
- net SW15: now reaches MX13.2 (ROW)
- net SW15: now also U3.17 (GPIO14)
- net SW8: now reaches MX8.2 (ROW)
- net SW8: now also U3.9 (GPIO7)
- net SW9: now reaches MX9.2 (ROW)
- net SW9: now also U3.11 (GPIO8)
- net SW2: now reaches MX2.2 (ROW)
- net SW2: now also U3.3 (GPIO1)
- net SW11: now reaches MX14.2 (ROW)
- net SW11: now also U3.13 (GPIO10)
- net SW5: now reaches MX5.2 (ROW)
- net SW5: now also U3.6 (GPIO4)
- net SW6: now reaches MX6.2 (ROW)
- net SW6: now also U3.7 (GPIO5)
- net SW7: now reaches MX7.2 (ROW)
- net SW7: now also U3.8 (GPIO6)
- net SW4: now reaches MX4.2 (ROW)
- net SW4: now also U3.5 (GPIO3)
- net SW13: now reaches MX11.2 (ROW)
- net SW13: now also U3.15 (GPIO12)
- net SW14: now reaches MX12.2 (ROW)
- net SW14: now also U3.16 (GPIO13)
- net SW10: now reaches MX10.2 (ROW)
- net SW10: now also U3.12 (GPIO9)
- new net: D5.2 (DOUT), D6.4 (DIN)
- new net: D4.2 (DOUT), D5.4 (DIN)
- new net: R6.2, U3.46 (USB_DM)
- new net: D1.4 (DIN), U3.41 (GPIO29_ADC3)
- new net: R5.2, U3.47 (USB_DP)
- new net: C5.1, R1.1, Y1.4
- new net: D1.2 (DOUT), D2.4 (DIN)
- new net: D2.2 (DOUT), D3.4 (DIN)
- new net: D3.2 (DOUT), D4.4 (DIN)
- new net +1V1: C6.2, C7.2, U3.23 (DVDD), U3.45 (VREG_VOUT), U3.50 (DVDD)
- new net +3V3: C10.2, C11.2, C12.2, C3.1, C8.2, C9.2, D1.1 (VDD), D2.1 (VDD), D3.1 (VDD), D4.1 (VDD), D5.1 (VDD), D6.1 (VDD), R2.2, R4.2, U1.2 (VO), U3.1 (IOVDD), U3.10 (IOVDD), U3.22 (IOVDD), U3.33 (IOVDD), U3.42 (IOVDD), U3.43 (ADC_AVDD), U3.44 (VREG_IN), U3.48 (USB_VDD), U3.49 (IOVDD)
- new net 3V3: C1.2, U2.8 (VCC)
- new net BOOT: R3.1, SW1.1
- new net DN: J1.2 (Pin_2), R6.1
- new net DP: J1.3 (Pin_3), R5.1
- new net QSPI_SCLK: U2.6 (CLK), U3.52 (QSPI_SCLK)
- new net QSPI_SD0: U2.5 (DI), U3.53 (QSPI_SD0)
- new net QSPI_SD1: U2.2 (DO), U3.55 (QSPI_SD1)
- new net QSPI_SD2: U2.3 (WP), U3.54 (QSPI_SD2)
- new net QSPI_SD3: U2.7 (HOLD), U3.51 (QSPI_SD3)
- new net QSPI_SS_N: R2.1, R3.2, U2.1 (CS), U3.56 (QSPI_SS)
- new net RUN: R4.1, SW2.1, U3.26 (RUN)
- new net VBUS: C2.1, J1.1 (Pin_1), U1.3 (VI)
- new net XIN: C4.1, U3.20 (XIN), Y1.1
- new net XOUT: R1.2, U3.21 (XOUT)
- no-connect marks 0 -> 18
Other:
- moved on the sheet: MX1, MX10, MX11, MX12, MX13, MX14, MX15, MX2, MX3, MX4, MX5, MX6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
